File: eagle/VCCS_Unit/VCCS_Unit.brd (EAGLE design)
At the start: 70.8 x 45.7 mm, 20 parts, among them IC1 OPA2134P, T1 2SC1815-GR, T2 2SC1815-GR, T3 2SA1015-GR, T4 2SA1015-GR

Commit message: Updated: the eagle files
Parts:
- moved LED1 2.54 mm to (34.3, 15.2)
- moved T1 2.54 mm to (27.9, 35.6)
- moved T4 2.54 mm to (58.4, 17.8)
Routing:
- net GND: track 0.00 -> 133.7 mm
- net VCC: track 0.00 -> 99.7 mm, vias 0 -> 2
- net N$9: track 0.00 -> 35.1 mm
- net N$10: track 0.00 -> 17.8 mm, vias 0 -> 2
- net N$8: track 0.00 -> 17.8 mm
- net N$7: track 0.00 -> 13.8 mm
- net N$4: track 0.00 -> 12.7 mm
- net N$6: track 0.00 -> 11.2 mm, vias 0 -> 2
- net N$5: track 0.00 -> 11.2 mm
- net N$3: track 0.00 -> 8.67 mm
- net N$1: track 0.00 -> 5.08 mm
- net N$2: track 0.00 -> 5.08 mm
- net N$11: track 0.00 -> 3.59 mm
